Commit message: map and scan working

File: src/navvis_description/urdf/robot.xacro (robot description, xacro)
@@ -17,82 +17,4 @@
         </collision>
     </link>
-    <!--
-    <joint name="base_laser_vert_bottom_joint" type="fixed">
-        <parent link="base" />
-        <child link="laser_vert_bottom" />
-        <origin xyz="0.3158 -0.0021 0.5100" rpy="3.1355 -1.3045 0.0025" />
-    </joint>
-    <link name="laser_vert_bottom">
-        <visual>
-            <origin xyz="0.0 0.0 0.0" rpy="0.0 0.0 0.0" />
-            <geometry>
-                <box size="0.062 0.062 0.087" />
-            </geometry>
-        </visual>
-        <collision>
-            <origin xyz="0.0 0.0 0.0" rpy="0.0 0.0 0.0" />
-            <geometry>
-                <box size="0.062 0.062 0.087" />
-            </geometry>
-        </collision>
-    </link>
-    <joint name="laser_vert_top_right_joint" type="fixed">
-        <parent link="base" />
-        <child link="laser_vert_top_right" />
-        <origin xyz="0.2978 -0.145 1.8451" rpy="-1.8451 0.6313 -1.9377" />
-    </joint>
-    <link name="laser_vert_top_right">
-        <visual>
-            <origin xyz="0.0 0.0 0.0" rpy="0.0 0.0 0.0" />
-            <geometry>
-                <box size="0.062 0.062 0.087" />
-            </geometry>
-        </visual>
-        <collision>
-            <origin xyz="0.0 0.0 0.0" rpy="0.0 0.0 0.0" />
-            <geometry>
-                <box size="0.062 0.062 0.087" />
-            </geometry>
-        </collision>
-    </link>
-    <joint name="laser_vert_top_left_joint" type="fixed">
-        <parent link="base" />
-        <child link="laser_vert_top_left" />
-        <origin xyz="0.2997 0.1531 1.8443" rpy="1.1780 0.6198 1.9560" />
-    </joint>
-    <link name="laser_vert_top_left">
-        <visual>
-            <origin xyz="0.0 0.0 0.0" rpy="0.0 0.0 0.0" />
-            <geometry>
-                <box size="0.062 0.062 0.087" />
-            </geometry>
-        </visual>
-        <collision>
-            <origin xyz="0.0 0.0 0.0" rpy="0.0 0.0 0.0" />
-            <geometry>
-                <box size="0.062 0.062 0.087" />
-            </geometry>
-        </collision>
-    </link>
-    <joint name="laser_horiz_joint" type="fixed">
-        <parent link="base" />
-        <child link="laser_horiz" />
-        <origin xyz="0.2325 0.0001 1.9201" rpy="-0.00120 0.1146 -0.0015" />
-    </joint>
-    <link name="laser_horiz">
-        <visual>
-            <origin xyz="0.0 0.0 0.0" rpy="0.0 0.0 0.0" />
-            <geometry>
-                <cylinder radius="0.052" length="0.072"/>
-            </geometry>
-        </visual>
-        <collision>
-            <origin xyz="0.0 0.0 0.0" rpy="0.0 0.0 0.0" />
-            <geometry>
-                <cylinder radius="0.052" length="0.072"/>
-            </geometry>
-        </collision>
-    </link>
-    -->
     <!-- XACRO Macro definition block to add around the wheel link and joint !-->
     <xacro:macro name="xacro_name" params="side reflect">
